Commit message: Fix Titati joint axes and align control defaults

File: new_titati/rl_sar/src/robots/titati_description/urdf/titati_description.urdf (robot description, URDF)
Before this commit: robot titati_description, 23 links, 22 joints
Joints:
- joint FR_foot_joint: axis 0 1 0 -> 0 -1 0
- joint RL_calf_joint: axis 0 1 0 -> 0 -1 0; limit lower=0.916297857297 upper=2.69653369433 effort=55 velocity=28.6 -> lower=-2.69653369433 upper=-0.916297857297 effort=55 velocity=28.6
- joint RL_foot_joint: axis 0 1 0 -> 0 -1 0
- joint RL_thigh_joint: axis 0 1 0 -> 0 -1 0; limit lower=-4.18879020479 upper=1.0471975512 effort=55 velocity=28.6 -> lower=-1.0471975512 upper=4.18879020479 effort=55 velocity=28.6
- joint RR_calf_joint: axis 0 1 0 -> 0 -1 0; limit lower=0.916297857297 upper=2.69653369433 effort=55 velocity=28.6 -> lower=-2.69653369433 upper=-0.916297857297 effort=55 velocity=28.6
- joint RR_foot_joint: axis 0 1 0 -> 0 -1 0
- joint RR_thigh_joint: axis 0 1 0 -> 0 -1 0; limit lower=-4.18879020479 upper=1.0471975512 effort=55 velocity=28.6 -> lower=-1.0471975512 upper=4.18879020479 effort=55 velocity=28.6
